Commit message: Still trying to get a good policy. Need to play with the observation space some more...

File: assets/urdf/Core.urdf (robot description, URDF)
Before this commit: robot Core, 7 links, 6 joints
Links:
- link Connector_1: geometry collision sphere radius=0.0025; visual sphere radius=0.0025
- link Connector_2: geometry collision sphere radius=0.0025; visual sphere radius=0.0025
- link Connector_3: geometry collision sphere radius=0.0025; visual sphere radius=0.0025
- link Connector_4: geometry collision sphere radius=0.0025; visual sphere radius=0.0025
- link Connector_5: geometry collision sphere radius=0.0025; visual sphere radius=0.0025
- link Connector_6: geometry collision sphere radius=0.0025; visual sphere radius=0.0025
- link Core: geometry collision sphere radius=0.005; visual sphere radius=0.005
Joints:
- joint $fixed_Core_Connector_1: origin xyz=0 0.01 0 rpy=0 0 0 -> xyz=0 0.005 0 rpy=0 0 0
- joint $fixed_Core_Connector_2: origin xyz=0 -0.01 0 rpy=0 0 0 -> xyz=0 -0.005 0 rpy=0 0 0
- joint $fixed_Core_Connector_3: origin xyz=0 0 0.01 rpy=0 0 0 -> xyz=0 0 0.005 rpy=0 0 0
- joint $fixed_Core_Connector_4: origin xyz=0 0 -0.01 rpy=0 0 0 -> xyz=0 0 -0.005 rpy=0 0 0
- joint $fixed_Core_Connector_5: origin xyz=0.01 0 0 rpy=0 0 0 -> xyz=0.005 0 0 rpy=0 0 0
- joint $fixed_Core_Connector_6: origin xyz=-0.01 0 0 rpy=0 0 0 -> xyz=-0.005 0 0 rpy=0 0 0

File: assets/urdf/core.xacro (robot description, xacro)
@@ -13,7 +13,7 @@
     <xacro:property name="Purple" value="0.8 0.1 0.8 1" />
     <!-- Physical Properties -->
-    <xacro:property name="CoreSize" value="0.01" />
-    <xacro:property name="ConnectorSize" value="0.005" />
-    <xacro:property name="ConnectionDist" value="0.01" />
+    <xacro:property name="CoreSize" value="0.005" />
+    <xacro:property name="ConnectorSize" value="0.0025" />
+    <xacro:property name="ConnectionDist" value="0.005" />
     <!-- Color Definitions-->
     <xacro:macro name="Mat" params="cname color">
